Commit message: Create custom Gazebo plugin for /cmd_vel-controlled differential drive
- Create custom_plugins package
- Add diff_drive_plugin.cpp to define custom Gazebo C++ plugin and implement kinematics
- Modify robot.urdf.xacro to adjust mass values, set friction coefficients for caster, reorient wheels for correct differential drive behaviour, and load the custom plugin
- Update .gitignore to ignore compile_commands.json

File: src/diff_drive_robot_description/urdf/robot.urdf.xacro (robot description, xacro)
@@ -5,10 +5,11 @@
     <xacro:property name="CHASSIS_WIDTH" value="0.10"/>  <!-- Along y axis -->
     <xacro:property name="CHASSIS_HEIGHT" value="0.10"/>  <!-- Along z axis -->
-    <xacro:property name="CHASSIS_MASS" value="0.5"/>
+    <xacro:property name="CHASSIS_MASS" value="2.0"/>
     <!-- Driven wheel constants with offset from chassis included in each joint origin -->
     <xacro:property name="DRIVEN_WHEEL_RADIUS" value="0.03"/>
     <xacro:property name="DRIVEN_WHEEL_WIDTH" value="0.015"/>
+    <xacro:property name="DRIVEN_WHEEL_OFFSET" value="0.01"/>
     <xacro:property name="DRIVEN_WHEEL_JOINT_X" value="${-CHASSIS_LENGTH / 4}"/>
-    <xacro:property name="DRIVEN_WHEEL_JOINT_Y_ABS" value="${CHASSIS_WIDTH / 2 + 0.01}"/>  <!-- Use as +ve for LHS and -ve for RHS -->
+    <xacro:property name="DRIVEN_WHEEL_JOINT_Y_ABS" value="${CHASSIS_WIDTH / 2 + DRIVEN_WHEEL_OFFSET}"/>  <!-- Use as +ve for LHS and -ve for RHS -->
     <xacro:property name="DRIVEN_WHEEL_JOINT_Z" value="${-CHASSIS_HEIGHT / 2}"/>
     <xacro:property name="DRIVEN_WHEEL_MASS" value="0.1"/>
@@ -59,5 +60,5 @@
         </xacro:if>
         <xacro:property name="joint_y" value="${sign * DRIVEN_WHEEL_JOINT_Y_ABS}"/>
-        <xacro:property name="joint_roll" value="${-sign * (math.pi / 2)}"/>  <!-- Orient the wheel correctly -->
+        <xacro:property name="joint_roll" value="${-math.pi / 2}"/>  <!-- Orient the wheel correctly for differential drive kinematics -->
         <!-- Driven wheel -->
         <link name="${prefix}_wheel_link">
@@ -137,5 +138,18 @@
         <parent link="chassis_link"/>
         <child link="caster_link"/>
-        <origin xyz="${CASTER_JOINT_X} 0 ${CASTER_JOINT_Z}" rpy="${math.pi / 2} 0 0"/>
+        <origin xyz="${CASTER_JOINT_X} 0 ${CASTER_JOINT_Z}" rpy="${-math.pi / 2} 0 0"/>
     </joint>
+    <gazebo reference="caster_link">
+        <mu1 value="0.001"/>
+        <mu2 value="0.001"/>
+    </gazebo>
+    <!-- Use custom differential drive kinematics plugin with driven wheel joint names as parameters -->
+    <gazebo>
+        <plugin name="custom::DiffDrivePlugin" filename="libCustomDiffDrivePlugin.so">
+            <left_wheel_joint_name>chassis_to_left_wheel_joint</left_wheel_joint_name>
+            <right_wheel_joint_name>chassis_to_right_wheel_joint</right_wheel_joint_name>
+            <wheel_radius>${DRIVEN_WHEEL_RADIUS}</wheel_radius>
+            <wheels_separation>${2 * DRIVEN_WHEEL_JOINT_Y_ABS}</wheels_separation>
+        </plugin>
+    </gazebo>
 </robot>

Commit message: Implement ros2_control differential drive using /cmd_vel input
- Create custom_control package
- Add controllers.yaml for controller_manager, joint_state_broadcaster, and diff_drive_controller parameters
- Add twist_to_twist_stamped.cpp node: subscribe to /cmd_vel, convert Twist to TwistStamped, and publish to /diff_drive_controller/cmd_vel
- Add controller.launch.py to spawn joint_state_broadcaster and diff_drive_controller and run twist_to_twist_stamped node
- Add simulate_control.launch.py to launch controller.launch.py and then simulate.launch.py
- Modify robot.urdf.xacro to optionally define transmission, ros2_control, and Gazebo control plugin tags based on controllers_config_path argument
- Modify simulate.launch.py to accept launch arguments: controllers_config_path (passed to xacro command) and run_sim (control whether simulation starts running or paused)

File: src/diff_drive_robot_description/urdf/robot.urdf.xacro (robot description, xacro)
@@ -1,4 +1,10 @@
 <?xml version="1.0"?>
 <robot name="diff_drive_robot" xmlns:xacro="http://www.ros.org/wiki/xacro">
+    <!-- Declare optional controllers config path which points to parameters YAML -->
+    <xacro:arg name="controllers_config_path" default=""/>
+    <!-- Promote it to a property for use in expressions -->
+    <xacro:property name="controllers_config_path" value="$(arg controllers_config_path)"/>
+    <!-- Define control-related tags only if path to the YAML is non-empty -->
+    <xacro:property name="use_control" value="${controllers_config_path != ''}"/>
     <!-- Chassis constants -->
     <xacro:property name="CHASSIS_LENGTH" value="0.15"/>  <!-- Along x axis -->
@@ -20,5 +26,5 @@
     <xacro:property name="CASTER_MASS" value="0.05"/>
     <!-- Constants for dynamics and motors -->
-    <xacro:property name="MAX_LINEAR_VELOCITY" value="1.0"/>  <!-- m/s - Use with wheel radius to calculate corresponding max angular velocity -->
+    <xacro:property name="MAX_LINEAR_VELOCITY" value="0.5"/>  <!-- m/s - Use with wheel radius to calculate corresponding max angular velocity -->
     <xacro:property name="MOTOR_MAX_TORQUE" value="0.5"/>  <!-- Nm -->
     <xacro:macro name="cylinder_inertial" params="radius length mass">
@@ -88,4 +94,14 @@
             <limit effort="${MOTOR_MAX_TORQUE}" velocity="${MAX_LINEAR_VELOCITY / DRIVEN_WHEEL_RADIUS}"/>
         </joint>
+        <xacro:if value="${use_control}">
+            <!-- Transmission for control -->
+            <transmission name="${prefix}_wheel_trans">
+                <type>transmission_interface/SimpleTransmission</type>
+                <joint name="chassis_to_${prefix}_wheel_joint"/>
+                <actuator name="${prefix}_motor">
+                    <mechanicalReduction>1</mechanicalReduction>
+                </actuator>
+            </transmission>
+        </xacro:if>
     </xacro:macro>
     <link name="base_link"/>
@@ -140,16 +156,40 @@
         <origin xyz="${CASTER_JOINT_X} 0 ${CASTER_JOINT_Z}" rpy="${-math.pi / 2} 0 0"/>
     </joint>
+    <!-- Set friction coefficients for driven wheels and caster -->
+    <gazebo reference="left_wheel_link">
+        <mu1 value="1.0"/>
+        <mu2 value="1.0"/>
+    </gazebo>
+    <gazebo reference="right_wheel_link">
+        <mu1 value="1.0"/>
+        <mu2 value="1.0"/>
+    </gazebo>
     <gazebo reference="caster_link">
         <mu1 value="0.001"/>
         <mu2 value="0.001"/>
     </gazebo>
-    <!-- Use custom differential drive kinematics plugin with driven wheel joint names as parameters -->
-    <gazebo>
-        <plugin name="custom::DiffDrivePlugin" filename="libCustomDiffDrivePlugin.so">
-            <left_wheel_joint_name>chassis_to_left_wheel_joint</left_wheel_joint_name>
-            <right_wheel_joint_name>chassis_to_right_wheel_joint</right_wheel_joint_name>
-            <wheel_radius>${DRIVEN_WHEEL_RADIUS}</wheel_radius>
-            <wheels_separation>${2 * DRIVEN_WHEEL_JOINT_Y_ABS}</wheels_separation>
-        </plugin>
-    </gazebo>
+    <xacro:if value="${use_control}">
+        <ros2_control name="GazeboSimSystem" type="system">
+            <hardware>
+                <plugin>gz_ros2_control/GazeboSimSystem</plugin>
+            </hardware>
+            <joint name="chassis_to_left_wheel_joint">
+                <command_interface name="velocity"/>
+                <state_interface name="velocity"/>
+                <state_interface name="position"/>
+            </joint>
+            <joint name="chassis_to_right_wheel_joint">
+                <command_interface name="velocity"/>
+                <state_interface name="velocity"/>
+                <state_interface name="position"/>
+            </joint>
+        </ros2_control>
+    </xacro:if>
+    <xacro:if value="${use_control}">
+        <gazebo>
+            <plugin filename="libgz_ros2_control-system.so" name="gz_ros2_control::GazeboSimROS2ControlPlugin">
+                <parameters>${controllers_config_path}</parameters>
+            </plugin>
+        </gazebo>
+    </xacro:if>
 </robot>

Commit message: Modularize URDF using multiple xacro files
- Add base.xacro: base link, chassis, and caster
- Add wheels.xacro: driven wheel macro with link, joint, and transmission
- Add macros.xacro: inertial tag macros for cylinder, cuboid, and sphere
- Add physics.xacro: constants, limits, and Gazebo parameters
- Add control.xacro: ros2_control and Gazebo control plugin
- Modify robot.urdf.xacro: include new xacro files in correct order

File: src/diff_drive_robot_description/urdf/robot.urdf.xacro (robot description, xacro)
@@ -7,189 +7,15 @@
     <!-- Define control-related tags only if path to the YAML is non-empty -->
     <xacro:property name="use_control" value="${controllers_config_path != ''}"/>
-    <!-- Chassis constants -->
-    <xacro:property name="CHASSIS_LENGTH" value="0.15"/>  <!-- Along x axis -->
-    <xacro:property name="CHASSIS_WIDTH" value="0.10"/>  <!-- Along y axis -->
-    <xacro:property name="CHASSIS_HEIGHT" value="0.10"/>  <!-- Along z axis -->
-    <xacro:property name="CHASSIS_MASS" value="2.0"/>
-    <!-- Driven wheel constants with offset from chassis included in each joint origin -->
-    <xacro:property name="DRIVEN_WHEEL_RADIUS" value="0.03"/>
-    <xacro:property name="DRIVEN_WHEEL_WIDTH" value="0.015"/>
-    <xacro:property name="DRIVEN_WHEEL_OFFSET" value="0.01"/>
-    <xacro:property name="DRIVEN_WHEEL_JOINT_X" value="${-CHASSIS_LENGTH / 4}"/>
-    <xacro:property name="DRIVEN_WHEEL_JOINT_Y_ABS" value="${CHASSIS_WIDTH / 2 + DRIVEN_WHEEL_OFFSET}"/>  <!-- Use as +ve for LHS and -ve for RHS -->
-    <xacro:property name="DRIVEN_WHEEL_JOINT_Z" value="${-CHASSIS_HEIGHT / 2}"/>
-    <xacro:property name="DRIVEN_WHEEL_MASS" value="0.1"/>
-    <!-- Caster constants (JOINT_Y left out because the joint is centered along chassis width) -->
-    <xacro:property name="CASTER_RADIUS" value="0.014"/>
-    <xacro:property name="CASTER_JOINT_X" value="${CHASSIS_LENGTH / 4}"/>
-    <xacro:property name="CASTER_JOINT_Z" value="${-CHASSIS_HEIGHT / 2 - (DRIVEN_WHEEL_RADIUS - CASTER_RADIUS)}"/> <!-- Caster will touch the ground and leave a gap from the chassis -->
-    <xacro:property name="CASTER_MASS" value="0.05"/>
-    <!-- Constants for dynamics and motors -->
-    <xacro:property name="MAX_LINEAR_VELOCITY" value="0.5"/>  <!-- m/s - Use with wheel radius to calculate corresponding max angular velocity -->
-    <xacro:property name="MOTOR_MAX_TORQUE" value="0.5"/>  <!-- Nm -->
-    <xacro:macro name="cylinder_inertial" params="radius length mass">
-        <inertial>
-            <mass value="${mass}"/>
-            <inertia
-                ixx="${(mass * (3 * radius**2 + length**2)) / 12}" ixy="0" ixz="0"
-                iyy="${(mass * (3 * radius**2 + length**2)) / 12}" iyz="0"
-                izz="${(mass * radius**2) / 2}"
-            />
-        </inertial>
-    </xacro:macro>
-    <xacro:macro name="box_inertial" params="length width height mass">
-        <inertial>
-            <mass value="${mass}"/>
-            <inertia
-                ixx="${(mass * (width**2 + height**2)) / 12}" ixy="0" ixz="0"
-                iyy="${(mass * (length**2 + height**2)) / 12}" iyz="0"
-                izz="${(mass * (length**2 + width**2)) / 12}"
-            />
-        </inertial>
-    </xacro:macro>
-    <xacro:macro name="sphere_inertial" params="radius mass">
-        <inertial>
-            <mass value="${mass}"/>
-            <inertia
-                ixx="${(2 / 5) * mass * radius**2}" ixy="0" ixz="0"
-                iyy="${(2 / 5) * mass * radius**2}" iyz="0"
-                izz="${(2 / 5) * mass * radius**2}"
-            />
-        </inertial>
-    </xacro:macro>
-    <xacro:macro name="driven_wheel" params="prefix">
-        <xacro:if value="${prefix == 'left'}">
-            <xacro:property name="sign" value="1"/>
-        </xacro:if>
-        <xacro:if value="${prefix == 'right'}">
-            <xacro:property name="sign" value="-1"/>
-        </xacro:if>
-        <xacro:property name="joint_y" value="${sign * DRIVEN_WHEEL_JOINT_Y_ABS}"/>
-        <xacro:property name="joint_roll" value="${-math.pi / 2}"/>  <!-- Orient the wheel correctly for differential drive kinematics -->
-        <!-- Driven wheel -->
-        <link name="${prefix}_wheel_link">
-            <xacro:cylinder_inertial radius="${DRIVEN_WHEEL_RADIUS}" length="${DRIVEN_WHEEL_WIDTH}" mass="${DRIVEN_WHEEL_MASS}"/>
-            <visual>
-                <origin xyz="0 0 0" rpy="0 0 0"/>
-                <geometry>
-                    <cylinder length="${DRIVEN_WHEEL_WIDTH}" radius="${DRIVEN_WHEEL_RADIUS}"/>
-                </geometry>
-                <material name="black">
-                    <color rgba="0 0 0 1.0"/>
-                </material>
-            </visual>
-            <collision>
-                <origin xyz="0 0 0" rpy="0 0 0"/>
-                <geometry>
-                    <cylinder length="${DRIVEN_WHEEL_WIDTH}" radius="${DRIVEN_WHEEL_RADIUS}"/>
-                </geometry>
-            </collision>
-        </link>
-        <!-- Join chassis to wheel with an offset to account for DC rotor -->
-        <joint name="chassis_to_${prefix}_wheel_joint" type="continuous">
-            <parent link="chassis_link"/>
-            <child link="${prefix}_wheel_link"/>
-            <origin xyz="${DRIVEN_WHEEL_JOINT_X} ${joint_y} ${DRIVEN_WHEEL_JOINT_Z}" rpy="${joint_roll} 0 0"/>
-            <axis xyz="0 0 1"/>
-            <limit effort="${MOTOR_MAX_TORQUE}" velocity="${MAX_LINEAR_VELOCITY / DRIVEN_WHEEL_RADIUS}"/>
-        </joint>
-        <xacro:if value="${use_control}">
-            <!-- Transmission for control -->
-            <transmission name="${prefix}_wheel_trans">
-                <type>transmission_interface/SimpleTransmission</type>
-                <joint name="chassis_to_${prefix}_wheel_joint"/>
-                <actuator name="${prefix}_motor">
-                    <mechanicalReduction>1</mechanicalReduction>
-                </actuator>
-            </transmission>
-        </xacro:if>
-    </xacro:macro>
-    <link name="base_link"/>
-    <!-- Main body of the robot -->
-    <link name="chassis_link">
-        <xacro:box_inertial length="${CHASSIS_LENGTH}" width="${CHASSIS_WIDTH}" height="${CHASSIS_HEIGHT}" mass="${CHASSIS_MASS}"/>
-        <visual>
-            <origin xyz="0 0 0" rpy="0 0 0"/>
-            <geometry>
-                <box size="${CHASSIS_LENGTH} ${CHASSIS_WIDTH} ${CHASSIS_HEIGHT}"/>
-            </geometry>
-            <material name="white">
-                <color rgba="1.0 1.0 1.0 1.0"/>
-            </material>
-        </visual>
-        <collision>
-            <origin xyz="0 0 0" rpy="0 0 0"/>
-            <geometry>
-                <box size="${CHASSIS_LENGTH} ${CHASSIS_WIDTH} ${CHASSIS_HEIGHT}"/>
-            </geometry>
-        </collision>
-    </link>
-    <joint name="base_to_chassis_joint" type="fixed">
-        <parent link="base_link"/>
-        <child link="chassis_link"/>
-        <origin xyz="${CHASSIS_LENGTH / 4} 0 ${CHASSIS_HEIGHT / 2 + DRIVEN_WHEEL_RADIUS}" rpy="0 0 0"/>
-    </joint>
-    <!-- Create driven wheel links and their joints to the chassis -->
-    <xacro:driven_wheel prefix="left"/>
-    <xacro:driven_wheel prefix="right"/>
-    <link name="caster_link">
-        <xacro:sphere_inertial radius="${CASTER_RADIUS}" mass="${CASTER_MASS}"/>
-        <visual>
-            <origin xyz="0 0 0" rpy="0 0 0"/>
-            <geometry>
-                <sphere radius="${CASTER_RADIUS}"/>
-            </geometry>
-            <material name="black">
-                <color rgba="0 0 0 1.0"/>
-            </material>
-        </visual>
-        <collision>
-            <origin xyz="0 0 0" rpy="0 0 0"/>
-            <geometry>
-                <sphere radius="${CASTER_RADIUS}"/>
-            </geometry>
-        </collision>
-    </link>
-    <joint name="chassis_to_caster_joint" type="fixed">
-        <parent link="chassis_link"/>
-        <child link="caster_link"/>
-        <origin xyz="${CASTER_JOINT_X} 0 ${CASTER_JOINT_Z}" rpy="${-math.pi / 2} 0 0"/>
-    </joint>
-    <!-- Set friction coefficients for driven wheels and caster -->
-    <gazebo reference="left_wheel_link">
-        <mu1 value="1.0"/>
-        <mu2 value="1.0"/>
-    </gazebo>
-    <gazebo reference="right_wheel_link">
-        <mu1 value="1.0"/>
-        <mu2 value="1.0"/>
-    </gazebo>
-    <gazebo reference="caster_link">
-        <mu1 value="0.001"/>
-        <mu2 value="0.001"/>
-    </gazebo>
+    <!-- Get physical constants and Gazebo physics tags -->
+     <xacro:include filename="physics.xacro"/>
+    <!-- Define base link, chassis, and caster -->
+    <xacro:include filename="base.xacro"/>
+    <!-- Get macro to define driven wheel links and their joints to the chassis -->
+    <xacro:include filename="wheels.xacro"/>
+    <xacro:driven_wheel prefix="left" use_control="${use_control}"/>
+    <xacro:driven_wheel prefix="right" use_control="${use_control}"/>
+    <!-- Define ros2_control tag and Gazebo control plugin if control is switched on -->
     <xacro:if value="${use_control}">
-        <ros2_control name="GazeboSimSystem" type="system">
-            <hardware>
-                <plugin>gz_ros2_control/GazeboSimSystem</plugin>
-            </hardware>
-            <joint name="chassis_to_left_wheel_joint">
-                <command_interface name="velocity"/>
-                <state_interface name="velocity"/>
-                <state_interface name="position"/>
-            </joint>
-            <joint name="chassis_to_right_wheel_joint">
-                <command_interface name="velocity"/>
-                <state_interface name="velocity"/>
-                <state_interface name="position"/>
-            </joint>
-        </ros2_control>
-    </xacro:if>
-    <xacro:if value="${use_control}">
-        <gazebo>
-            <plugin filename="libgz_ros2_control-system.so" name="gz_ros2_control::GazeboSimROS2ControlPlugin">
-                <parameters>${controllers_config_path}</parameters>
-            </plugin>
-        </gazebo>
+        <xacro:include filename="control.xacro"/>
     </xacro:if>
 </robot>
