Commit message: Configure controller acceleration limits and update robot chassis mass
- Modify controllers.yaml to set linear max and min acceleration limits of 2.0 and -1.5 respectively
- Modify base.xacro to increase chassis mass from 2.0 to 4.75

File: src/diff_drive_robot_description/urdf/base.xacro (robot description, xacro)
@@ -7,5 +7,5 @@
     <xacro:property name="CHASSIS_WIDTH" value="0.10"/>  <!-- Along y axis -->
     <xacro:property name="CHASSIS_HEIGHT" value="0.10"/>  <!-- Along z axis -->
-    <xacro:property name="CHASSIS_MASS" value="2.0"/>
+    <xacro:property name="CHASSIS_MASS" value="4.75"/>
     <!-- Caster constants (JOINT_Y left out because the joint is centered along chassis width) -->
     <xacro:property name="CASTER_RADIUS" value="0.014"/>
