Commit message: Create more flexible robot description, display, simulation, and control for real/sim workflows
- Add 'hardware_type' xacro argument to URDF and expose it as launch argument, which can disable control or switch between hardware interface types
- Modularize creation of robot_state_publisher node with launch script for smoother changes between real/sim workflows
- Add mandatory 'use_sim_time' launch argument to description publisher, display, and controller launch scripts for consistent time behaviour
- Modify display launch to create joint_state_publisher_gui only if use_sim_time is 'false', which avoids redundancy when Rviz2 is running during simulation
- Remove redundant controller_manager block from controller YAML configuration and rename file to reflect single-controller intent
- Conditionally create ros2_control_node in controller launch to handle manual (real) or Gazebo-internal (simulation) controller_manager creation

File: src/diff_drive_robot_description/urdf/control.xacro (robot description, xacro)
@@ -1,7 +1,12 @@
 <robot xmlns:xacro="http://www.ros.org/wiki/xacro">
     <!-- Define ros2_control hardware, command, and state interfaces -->
-    <ros2_control name="GazeboSimSystem" type="system">
+    <ros2_control name="RobotSystem" type="system">
         <hardware>
-            <plugin>gz_ros2_control/GazeboSimSystem</plugin>
+            <xacro:if value="${hardware_type == 'real'}">
+                <plugin>mock_components/GenericSystem</plugin>
+            </xacro:if>
+            <xacro:if value="${hardware_type == 'simulated'}">
+                <plugin>gz_ros2_control/GazeboSimSystem</plugin>
+            </xacro:if>
         </hardware>
         <joint name="chassis_to_left_wheel_joint">
@@ -16,9 +21,11 @@
         </joint>
     </ros2_control>
-    <!-- Specify Gazebo control plugin -->
-    <gazebo>
-        <plugin filename="libgz_ros2_control-system.so" name="gz_ros2_control::GazeboSimROS2ControlPlugin">
-            <parameters>${controllers_config_path}</parameters>
-        </plugin>
-    </gazebo>
+    <xacro:if value="${hardware_type == 'simulated'}">
+        <!-- Specify Gazebo control plugin -->
+        <gazebo>
+            <plugin filename="libgz_ros2_control-system.so" name="gz_ros2_control::GazeboSimROS2ControlPlugin">
+                <parameters>${controller_config_path}</parameters>
+            </plugin>
+        </gazebo>
+    </xacro:if>
 </robot>

File: src/diff_drive_robot_description/urdf/robot.urdf.xacro (robot description, xacro)
@@ -1,10 +1,31 @@
 <?xml version="1.0"?>
 <robot name="diff_drive_robot" xmlns:xacro="http://www.ros.org/wiki/xacro">
-    <!-- Declare optional controllers config path which points to parameters YAML -->
-    <xacro:arg name="controllers_config_path" default=""/>
-    <!-- Promote it to a property for use in expressions -->
-    <xacro:property name="controllers_config_path" value="$(arg controllers_config_path)"/>
-    <!-- Define control-related tags only if path to the YAML is non-empty -->
-    <xacro:property name="use_control" value="${controllers_config_path != ''}"/>
+    <!--
+    Declare optional controller config path which points to parameters YAML. Default value
+    of '' disables control
+    -->
+    <xacro:arg name="controller_config_path" default=""/>
+    <!--
+    Declare optional hardware type ('real' or 'simulated') to signal which hardware interface
+    should be used. Default value of '' disables control
+    -->
+    <xacro:arg name="hardware_type" default=""/>
+    <!-- Promote arguments to properties for use in expressions -->
+    <xacro:property name="controller_config_path" value="$(arg controller_config_path)"/>
+    <xacro:property name="hardware_type" value="$(arg hardware_type)"/>
+    <!-- Validate hardware type value -->
+    <xacro:if value="${hardware_type not in ['', 'real', 'simulated']}">
+        <!--
+        Use undefined macro to raise error during xacro processing and signal that hardware
+        type is invalid -->
+        <xacro:invalid_hardware_type/>
+    </xacro:if>
+    <!--
+    Enable control and define relevant tags only if controller YAML path is non-empty and
+    hardware type is both non-empty and valid -->
+    <xacro:property
+        name="use_control"
+        value="${controller_config_path != '' and hardware_type in ['real', 'simulated']}"
+    />
     <!-- Get physical constants and Gazebo physics tags -->
      <xacro:include filename="physics.xacro"/>
